File: control_board/control_board.kicad_pcb (KiCad board)
At the start: 2 copper layers, 66 x 76.2 mm, 22 parts, among them J1 jst xh 2, J2 jst xh 2, J3 jst xh 2, J4 jst xh 2, J5 jst xh 2, J6 440052-3, J7 440052-3, J8 pwr_in, J9 jst xh 2, Q1 BUK9832-55A_CUX

Commit message: finish control board
Parts:
- U2: footprint esp32-gateway:polulu -> esp32-gateway:polulu-durin
- moved R8 24.8 mm to (114.3, 58.4), turned to 0 degrees
- moved R2 7.62 mm to (114.3, 61.0)
- moved R5 5.08 mm to (114.3, 66.0)
- moved R4 5.08 mm to (114.3, 68.6)
- moved J7 5.04 mm to (88.8, 93.9), turned to 180 degrees
- moved J6 5.00 mm to (88.8, 102.2), turned to 180 degrees
- moved Q1 4.32 mm to (98.5, 77.9)
- moved U2 2.57 mm to (81.5, 81.3)
- moved R3 2.54 mm to (114.3, 63.5)
Connections:
- R2 pad 2: /LED1 -> /LED3
- R3 pad 2: /LED2 -> /LED1
- R4 pad 2: /LED3 -> /LED2
- U1 pad 10: unconnected-(U1-IO15-Pad10) -> /BUTTON
- U1 pad 16: /BUTTON -> unconnected-(U1-I35-Pad16)
- U1 pad 6: /LED1 -> /LED2
- U1 pad 7: /LED2 -> /LED4
- U1 pad 8: /LED3 -> /LED1
- U1 pad 9: /LED4 -> /LED3
- U2 pad 2: unconnected-(U2-nSHDN-Pad2) -> +12V
- U2 pad 3: +12V -> Earth
Routing:
- net +3V3: track 0.00 -> 87.9 mm, vias 0 -> 3
- net /SERVO_TRX: track 0.00 -> 87.3 mm, vias 0 -> 1
- net Net-(J1-Pin_2): track 0.00 -> 48.3 mm, vias 0 -> 1
- net /BUTTON: track 0.00 -> 46.9 mm, vias 0 -> 1
- net /FAN_EN: track 0.00 -> 41.6 mm, vias 0 -> 2
- net Net-(J5-Pin_2): track 0.00 -> 37.3 mm, vias 0 -> 1
- net Net-(J4-Pin_2): track 0.00 -> 33.9 mm, vias 0 -> 1
- net Net-(J2-Pin_2): track 0.00 -> 29.5 mm, vias 0 -> 1
- net Net-(J3-Pin_2): track 0.00 -> 26.0 mm, vias 0 -> 1
- net /FAN_GND: track 0.00 -> 24.8 mm, vias 0 -> 1
- net +12V: track 0.00 -> 16.8 mm
- net Net-(U1-IO32): track 0.00 -> 4.16 mm
- net /LED2: track 0.00 -> 4.16 mm
- net /LED1: track 0.00 -> 4.16 mm
- net /LED3: track 0.00 -> 4.16 mm
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- added copper zone on F.Cu, net +12V
- added copper zone on F.Cu, net +3V3
