File: control_board/control_board.kicad_sch (KiCad schematic)
At the start: 21 parts, among them J1 jst xh 2, J2 jst xh 2, J3 jst xh 2, J4 jst xh 2, J5 jst xh 2, J6 440052-3, J7 440052-3, J8 pwr_in, J9 jst xh 2, Q1 BUK9832-55A_CUX

Commit message: finish control board
Parts:
- removed U2: ~, esp32-gateway:polulu, symbol esp32-gateway:polulu
- added U2: ~, esp32-gateway:polulu-durin, symbol esp32-gateway:polulu-durin
Connections:
- net +12V: now also U2.2 (IN)
- net +3V3: now also U2.5 (OUT)
- net BUTTON: now also U1.10 (IO15); no longer U1.16 (I35)
- net Earth: now also U2.3 (GND), U2.4 (GND)
- net LED1: now also R3.2, U1.8 (IO13); no longer R2.2, U1.6 (IO4)
- net LED2: now also R4.2, U1.6 (IO4); no longer R3.2, U1.7 (IO12)
- net LED3: now also R2.2, U1.9 (IO14); no longer R4.2, U1.8 (IO13)
- net LED4: now also U1.7 (IO12); no longer U1.9 (IO14)
- no-connect marks 10 -> 9
